File: HW_PCB/LaMano/Blue_pill/Blue_pill.kicad_pcb (KiCad board)
At the start: 2 copper layers, 44 x 32.6 mm, 32 parts, among them J1 V_Battery, J2 STLINK, J5 MPU6050, J6 NRF24, J7 UART, J8 PINHD_1x3_Male, SW1 SW_DPST_x2, SW2 SW_DPST_x2, U1 STM32F103C8Tx, U2 AMS1117-3.3, X1 Crystal

Commit message: fix: ConnectLaMano Veins
Parts:
- moved R1 51.9 mm to (56.2, 119.5)
- moved C3 51.8 mm to (61.4, 119.5)
- moved C1 51.8 mm to (45.6, 114.1)
- moved C6 51.8 mm to (43.1, 114.1)
- moved C9 51.8 mm to (48.0, 114.1)
- moved R8 51.8 mm to (77.7, 98.9)
- moved C4 51.8 mm to (53.1, 101.2)
- moved C5 51.8 mm to (44.4, 108.0)
- moved C7 51.8 mm to (72.3, 100.9)
- moved C8 51.8 mm to (72.3, 103.3)
- moved D1 51.8 mm to (44.1, 100.5)
- moved J5 51.8 mm to (49.2, 96.9)
- moved J6 51.8 mm to (73.9, 120.7)
- moved J7 51.8 mm to (61.7, 123.3)
- moved J8 51.8 mm to (50.3, 123.3)
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Routing:
- net GND: track 198.8 -> 232.7 mm, vias 2 -> 6
- net VCC: track 193.3 -> 219.4 mm, vias 3 -> 4
- net ADC2: track 38.8 -> 52.7 mm
- net VIN: track 16.4 -> 21.1 mm, vias 0 -> 1
- net SDA: track 14.6 -> 12.1 mm
- net NRST: track 26.6 -> 24.1 mm
- net Net-(U1-PB2): track 2.64 -> 4.65 mm
- net SWCLK: track 16.2 -> 18.0 mm, vias 0 -> 1
- net ADC1: track 11.0 -> 12.2 mm, vias 0 -> 1
- net TX: track 7.69 -> 8.87 mm, vias 0 -> 1
- net CE: track 18.9 -> 17.8 mm
- net SCK: track 13.2 -> 14.2 mm
- net CSN: track 17.1 -> 18.0 mm
- net RX: track 9.00 -> 8.30 mm, vias 0 -> 1
- net SW_LUZ: vias 0 -> 1
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Other:
- board size 44 x 32.6 mm -> 47 x 32.6 mm
